Commit message: checkpoint

File: custom_ws/src/togo_custom/togo_description/urdf/togo_description.urdf.xacro (robot description, xacro)
@@ -1,13 +1,92 @@
 <?xml version="1.0"?>
 <robot xmlns:xacro="http://www.ros.org/wiki/xacro">
-  <!-- Sim-only IMU for TOGO/Husky SLAM testing.
-       Clearpath's generated Phidgets entry creates the visual/link, but in
-       Gazebo the IMU topic was not published. Use a unique sensor name to
-       avoid colliding with any stock sensor named imu_0. -->
-  <gazebo reference="imu_0_link">
-    <sensor name="togo_imu_0" type="imu">
+  <!--
+    Simulated Seyond Robin W-style sensor package for Husky/TOGO testing.
+    This is intentionally a stable integration model, not a vendor-accurate
+    hardware driver simulation.
+    Public Robin W-style FOV target:
+      horizontal: 120 deg (-60 to +60)
+      vertical:    70 deg (-35 to +35)
+  -->
+  <link name="seyond_robin_w_link">
+    <visual>
+      <origin xyz="0 0 0" rpy="0 0 0"/>
+      <geometry>
+        <box size="0.16 0.10 0.08"/>
+      </geometry>
+      <material name="seyond_black">
+        <color rgba="0.02 0.025 0.03 1.0"/>
+      </material>
+    </visual>
+    <collision>
+      <origin xyz="0 0 0" rpy="0 0 0"/>
+      <geometry>
+        <box size="0.16 0.10 0.08"/>
+      </geometry>
+    </collision>
+    <inertial>
+      <origin xyz="0 0 0" rpy="0 0 0"/>
+      <mass value="0.8"/>
+      <inertia ixx="0.0011" ixy="0.0" ixz="0.0" iyy="0.0019" iyz="0.0" izz="0.0022"/>
+    </inertial>
+  </link>
+  <joint name="seyond_robin_w_mount_joint" type="fixed">
+    <parent link="base_link"/>
+    <child link="seyond_robin_w_link"/>
+    <origin xyz="0.30 0.0 0.42" rpy="0.0 0.0 0.0"/>
+  </joint>
+  <link name="seyond_robin_w_lidar_frame"/>
+  <joint name="seyond_robin_w_lidar_joint" type="fixed">
+    <parent link="seyond_robin_w_link"/>
+    <child link="seyond_robin_w_lidar_frame"/>
+    <origin xyz="0 0 0" rpy="0 0 0"/>
+  </joint>
+  <link name="seyond_robin_w_imu_frame"/>
+  <joint name="seyond_robin_w_imu_joint" type="fixed">
+    <parent link="seyond_robin_w_link"/>
+    <child link="seyond_robin_w_imu_frame"/>
+    <origin xyz="0 0 0" rpy="0 0 0"/>
+  </joint>
+  <gazebo reference="seyond_robin_w_lidar_frame">
+    <sensor name="seyond_robin_w_lidar" type="gpu_lidar">
+      <always_on>true</always_on>
+      <visualize>true</visualize>
+      <update_rate>15</update_rate>
+      <topic>/a300_0000/sensors/seyond_robin_w/scan</topic>
+      <gz_frame_id>seyond_robin_w_lidar_frame</gz_frame_id>
+      <lidar>
+        <scan>
+          <horizontal>
+            <samples>256</samples>
+            <resolution>1</resolution>
+            <min_angle>-1.0471975512</min_angle>
+            <max_angle>1.0471975512</max_angle>
+          </horizontal>
+          <vertical>
+            <samples>32</samples>
+            <resolution>1</resolution>
+            <min_angle>-0.6108652382</min_angle>
+            <max_angle>0.6108652382</max_angle>
+          </vertical>
+        </scan>
+        <range>
+          <min>0.2</min>
+          <max>80.0</max>
+          <resolution>0.02</resolution>
+        </range>
+        <noise>
+          <type>gaussian</type>
+          <mean>0.0</mean>
+          <stddev>0.005</stddev>
+        </noise>
+      </lidar>
+    </sensor>
+  </gazebo>
+  <gazebo reference="seyond_robin_w_imu_frame">
+    <sensor name="seyond_robin_w_imu" type="imu">
       <always_on>true</always_on>
       <update_rate>100</update_rate>
-      <topic>/a300_0000/sensors/imu_0/data</topic>
+      <topic>/a300_0000/sensors/seyond_robin_w/imu</topic>
+      <gz_frame_id>seyond_robin_w_imu_frame</gz_frame_id>
       <imu>
         <angular_velocity>
@@ -17,7 +96,7 @@
         </angular_velocity>
         <linear_acceleration>
-          <x><noise type="gaussian"><mean>0.0</mean><stddev>0.01</stddev></noise></x>
-          <y><noise type="gaussian"><mean>0.0</mean><stddev>0.01</stddev></noise></y>
-          <z><noise type="gaussian"><mean>0.0</mean><stddev>0.01</stddev></noise></z>
+          <x><noise type="gaussian"><mean>0.0</mean><stddev>0.005</stddev></noise></x>
+          <y><noise type="gaussian"><mean>0.0</mean><stddev>0.005</stddev></noise></y>
+          <z><noise type="gaussian"><mean>0.0</mean><stddev>0.005</stddev></noise></z>
         </linear_acceleration>
       </imu>

Commit message: more reliable frontend

File: custom_ws/src/togo_custom/togo_description/urdf/togo_description.urdf.xacro (robot description, xacro)
@@ -46,5 +46,6 @@
     <parent link="seyond_robin_w_link"/>
     <child link="seyond_robin_w_imu_frame"/>
-    <origin xyz="0 0 0" rpy="0 0 0"/>
+    <!-- Known LiDAR-to-IMU offset for extrinsic self-calibration tests. -->
+    <origin xyz="0.15 -0.05 0.08" rpy="0 0 0"/>
   </joint>
   <gazebo reference="seyond_robin_w_lidar_frame">
